File: High Resolution Multislope converter-modified rev 2.kicad_pcb (KiCad board)
At the start: 2 copper layers, 100 x 100 mm, 260 parts, among them J1 UART, J2 Input, J3 ICSP6, J4 ISCP10, J5 Power, Q1 BC856, Q2 BC847, Q3 BC856, Q4 BC856, Q5 BC856, Q6 BC856, Q7 BC847, Q8 BC847, Q9 BC856, U1 OPA172, U10 LM393, U11 OPA145, U12 OPA145, U13 MCP6002, U14 7815, U15 7915, U16 LTC2057, U17 74HC74, U18 OPA197, U19 OPA172, U2 OPA172, U20 DG419LDY, U202 MCP4921, U204 ADuM1201AR, U21 OP07CR, U3 7805, U4 NE5534D, U5 74LV4053, U6 LM399H, U7 DG408DJ, U8 OP07CR, U9 OP07CR, X1 16MHz

Commit message: Publish MiDi KiCad project, BOM and board views
Include the current schematic and PCB with portable project libraries,
schematic BOMs, Gerber/drill exports and the interactive PCB viewer.
Add colour PCB layer plots, four white-mask/black-silkscreen 3D views
and the assembled-board photograph.
Parts:
- added REF**: KiCAD Logo, Symbols:Symbol_KiCAD-Logo_CopperAndSilkScreenTop, F.Cu at (72.9, 83.8)
- added REF***: ESD-Logo_6.6x6mm_SilkScreen, Symbols:ESD-Logo_6.6x6mm_SilkScreen, F.Cu at (60.6, 92.1)
- added REF***: WEEE-Logo_4.2x6mm_SilkScreen, Symbols:WEEE-Logo_4.2x6mm_SilkScreen, F.Cu at (62.2, 83.1)
Routing:
- net /Analog_-15V: track 112.4 -> 112.9 mm
Other:
- outline, holes or cut-outs redrawn
- net class Default removed
- rule pad_to_mask_clearance: 0.02 -> 0
- board text added: "High resolution multi-slope ADC"
- board text added: "JLCJLCJLCJLC"
- board text added: "Kleinstein & Rerouter 2020"
- board text added: "github.com/Rerouter/Multislope-ADC-PCB minor modifications by Michael D."
